Commit message: GLM5.2 fixed.

File: urdf/Lite3.urdf (robot description, URDF)
Before this commit: robot Lite3, 17 links, 16 joints
Links:
- added link base_link, mass 0.001
- added link head_camera_depth_optical_frame, mass 0.001
- added link head_camera_link, mass 0.001
- added link head_camera_rgb_optical_frame, mass 0.001
- added link ultrasonic_front_link, mass 0.001
- added link ultrasonic_rear_link, mass 0.001
Joints:
- added joint TORSO_to_head_camera: type fixed, parent TORSO, child head_camera_link, origin xyz=0.18 0 0.18 rpy=0 0 0
- added joint TORSO_to_ultrasonic_front: type fixed, parent TORSO, child ultrasonic_front_link, origin xyz=0.25 0 0.05 rpy=0 0 0
- added joint TORSO_to_ultrasonic_rear: type fixed, parent TORSO, child ultrasonic_rear_link, origin xyz=-0.25 0 0.05 rpy=3.1415927 0 0
- added joint base_link_to_TORSO: type fixed, parent base_link, child TORSO, origin xyz=0 0 0 rpy=0 0 0
- added joint head_camera_to_depth_optical: type fixed, parent head_camera_link, child head_camera_depth_optical_frame, origin xyz=0 0 0 rpy=-1.5707963 0 -1.5707963
- added joint head_camera_to_rgb_optical: type fixed, parent head_camera_link, child head_camera_rgb_optical_frame, origin xyz=0 0 0 rpy=-1.5707963 0 -1.5707963

Commit message: LIVOX MID-360S adaptation.

File: urdf/Lite3.urdf (robot description, URDF)
Before this commit: robot Lite3, 23 links, 22 joints
Links:
- added link lidar_link, mass 0.001
Joints:
- added joint TORSO_to_lidar: type fixed, parent TORSO, child lidar_link, origin xyz=0 0 0.30 rpy=0 0 0
